Commit message: added robot description to robot

File: robo4_project/resource/demo.urdf (robot description, URDF)
Before this commit: robot /home/holly/ros2_ws/src/demo.urdf, 14 links, 13 joints
Links:
- removed link camera
- removed link panda_distance_sensor
Joints:
- removed joint panda_finger::left
- removed joint panda_finger::right
- removed joint panda_link7_camera_joint
- removed joint panda_link7_panda hand_joint
- removed joint panda_link7_panda_distance_sensor_joint
- added joint panda_finger_joint1: type prismatic, parent panda hand, child panda_rightfinger, origin xyz=-0.014101 0.005841 0.0584 rpy=0 0 -0.785398, axis 0.707107 -0.707107 0, limit lower=0 upper=0.04 effort=100 velocity=0.2
- added joint panda_finger_joint2: type prismatic, parent panda hand, child panda_leftfinger, origin xyz=0.028242 -0.019958 0.0584 rpy=0 0 -0.785398, axis -0.707107 0.707107 0, limit lower=0 upper=0.04 effort=100 velocity=0.2
- added joint panda_link7_panda_hand_joint: type fixed, parent panda_link7, child panda hand, origin xyz=0 0 0.107 rpy=0 0 0

Commit message: urdf update

File: robo4_project/resource/demo.urdf (robot description, URDF)
Before this commit: robot Panda, 12 links, 11 joints
Joints:
- removed joint base_link_solid_joint
- removed joint panda_finger_joint1
- removed joint panda_finger_joint2
- removed joint panda_joint1
- removed joint panda_joint2
- removed joint panda_joint3
- removed joint panda_joint4
- removed joint panda_joint5
- removed joint panda_joint6
- removed joint panda_joint7
- removed joint panda_link7_panda_hand_joint

Commit message: perfected urdf

File: robo4_project/resource/demo.urdf (robot description, URDF)
Before this commit: robot Panda, 12 links, 0 joints
Links:
- removed link panda hand
- added link panda_hand; collision box size=0.04 0.2 0.07; collision box size=0.057 0.055 0.01
Joints:
- added joint base_link_solid_joint: type fixed, parent base_link, child solid, origin xyz=-0.000005 0 -0.000272 rpy=-0.000003 0.00006 0
- added joint panda_link7_panda_hand_joint: type fixed, parent panda_link7, child panda_hand, origin xyz=0 0 0.107 rpy=0 0 0

Commit message: reverted back to panda.urdf

File: robo4_project/resource/demo.urdf (robot description, URDF)
Before this commit: robot Panda, 12 links, 2 joints
Joints:
- added joint panda_finger_joint1: type prismatic, parent panda_hand, child panda_rightfinger, origin xyz=-0.014101 0.005841 0.0584 rpy=0 0 -0.785398, axis 0.707107 -0.707107 0, limit lower=0 upper=0.04 effort=100 velocity=0.2
- added joint panda_finger_joint2: type prismatic, parent panda_hand, child panda_leftfinger, origin xyz=0.028242 -0.019958 0.0584 rpy=0 0 -0.785398, axis -0.707107 0.707107 0, limit lower=0 upper=0.04 effort=100 velocity=0.2
- added joint panda_joint1: type revolute, parent solid, child panda_link1, origin xyz=0 0 0.14 rpy=0 0 0.000051, axis 0 0 1, limit lower=-2.9671 upper=2.9671 effort=87 velocity=2.5
- added joint panda_joint2: type revolute, parent panda_link1, child panda_link2, origin xyz=0 0 0.193 rpy=-1.570796 0.220254 0, axis 0 0 1, limit lower=-1.8326 upper=1.8326 effort=87 velocity=2.5
- added joint panda_joint3: type revolute, parent panda_link2, child panda_link3, origin xyz=0 -0.195 0 rpy=1.570796 0.000282 0, axis 0 0 1, limit lower=-2.9671 upper=2.9671 effort=87 velocity=2.5
- added joint panda_joint4: type revolute, parent panda_link3, child panda_link4, origin xyz=0.0825 0 0.121 rpy=-1.570796 0.832446 -3.141592, axis 0.000001 0 1, limit lower=-3.1416 upper=-0.4 effort=87 velocity=2.5
- added joint panda_joint5: type revolute, parent panda_link4, child panda_link5, origin xyz=-0.0825 0.125 0 rpy=-1.570796 -0.000013 0, axis 0 0 1, limit lower=-2.9671 upper=2.9671 effort=12 velocity=3
- added joint panda_joint6: type revolute, parent panda_link5, child panda_link6, origin xyz=0 0 0.259 rpy=-1.570797 -0.61123 -3.141593, axis 0 0 1, limit lower=-0.0873 upper=3.8223 effort=12 velocity=3
- added joint panda_joint7: type revolute, parent panda_link6, child panda_link7, origin xyz=0.088 -0.058 0 rpy=1.570796 -0.789999 0, axis 0 0 1, limit lower=-2.9671 upper=2.9671 effort=12 velocity=3
